Commit message: modify urdf to set the joint mors as fixed

File: myGym/envs/robots/niryo_robot_description/urdf/ned2/niryo_ned2_gripper1_n_camera.urdf (robot description, URDF)
Before this commit: robot niryo_ned2, 14 links, 13 joints
Joints:
- joint gjoint_base_to_mors_1: type prismatic -> fixed
- joint gjoint_base_to_mors_2: type prismatic -> fixed

Commit message: edit collision filter

File: myGym/envs/robots/niryo_robot_description/urdf/ned2/niryo_ned2_gripper1_n_camera.urdf (robot description, URDF)
Before this commit: robot niryo_ned2, 14 links, 13 joints
Joints:
- joint gjoint_base_to_mors_1: type fixed -> prismatic
- joint gjoint_base_to_mors_2: type fixed -> prismatic
