Commit message: change plane 0.001 and cube_holes 0.02

File: myGym/envs/objects/assembly/urdf/cube_holes.urdf (robot description, URDF)
Before this commit: robot cube_holes, 1 links, 0 joints
Links:
- link baseLink: geometry collision mesh filename=../obj/cube_holes.obj scale=.0004 .0004 .0004; visual mesh filename=../obj/cube_holes.obj scale=.0004 .0004 .0004

Commit message: modify workspace and addin push task

File: myGym/envs/objects/assembly/urdf/cube_holes.urdf (robot description, URDF)
Before this commit: robot cube_holes, 1 links, 0 joints
Links:
- link baseLink: geometry collision mesh filename=../obj/cube_holes.obj scale=.001 .001 .001; visual mesh filename=../obj/cube_holes.obj scale=.001 .001 .001

File: myGym/envs/objects/storage/urdf/target.urdf (robot description, URDF)
Before this commit: robot target, 1 links, 0 joints
Links:
- link baseLink: geometry collision mesh filename=../obj/target.obj scale=0.0005 0.0005 0.0005; visual mesh filename=../obj/target.obj scale=0.0005 0.0005 0.0005
