Commit message: divide ned2 and ned2_gripper_camera

File: myGym/envs/robots/niryo_robot_description/urdf/ned2_ex/niryo_ned2.urdf (robot description, URDF)
Before this commit: robot niryo_ned2, 10 links, 9 joints
Links:
- removed link endeffector
- added link tool_link
Joints:
- removed joint hand_tool_gjoint
- removed joint rjoint_1
- removed joint rjoint_2
- removed joint rjoint_3
- removed joint rjoint_4
- removed joint rjoint_5
- removed joint rjoint_6
- added joint hand_tool_joint: type fixed, parent hand_link, child tool_link, origin xyz=0 0 0.0285 rpy=-1.5707963268 -1.5707963268 0
- added joint joint_1: type revolute, parent base_link, child shoulder_link, origin xyz=0 0 0.1013 rpy=0 0 -1.5707963268, axis 0 0 1, limit lower=-2.99987191833 upper=2.99987191833 effort=10.0 velocity=10.0
- added joint joint_2: type revolute, parent shoulder_link, child arm_link, origin xyz=0 0 0.065 rpy=1.5707963268 0 1.5707963268, axis 0 0 1, limit lower=-1.83259571459 upper=0.610167106497 effort=10.0 velocity=8.0
- added joint joint_3: type revolute, parent arm_link, child elbow_link, origin xyz=0.012 0.221 0 rpy=0 0 0, axis 0 0 1, limit lower=-1.34006379968 upper=1.57009819509 effort=7.0 velocity=8.0
- added joint joint_4: type revolute, parent elbow_link, child forearm_link, origin xyz=0.065 0.0325 0 rpy=0 1.5707963268 0, axis 0 0 1, limit lower=-2.09003177926 upper=2.09003177926 effort=7.0 velocity=2.0
- added joint joint_5: type revolute, parent forearm_link, child wrist_link, origin xyz=0 0 0.17 rpy=3.14159265359 -1.5707963268 3.14159265359, axis 0 0 1, limit lower=-1.92003671012 upper=1.92282923692 effort=6.0 velocity=2.0
- added joint joint_6: type revolute, parent wrist_link, child hand_link, origin xyz=0.0197 0.00925 0 rpy=0 1.5707963268 0, axis 0 0 1, limit lower=-2.53002928369 upper=2.53002928369 effort=5.0 velocity=2.0
