Commit message: use cube and modify target

File: myGym/envs/objects/geometric/urdf/cube.urdf (robot description, URDF)
Before this commit: robot cube.urdf, 1 links, 0 joints
Links:
- link baseLink: mass 0.113 -> 1e-4; geometry collision mesh filename=./obj/cube.obj scale=.0004 .0004 .0004; visual mesh filename=./obj/cube.obj scale=.0004 .0004 .0004

File: myGym/envs/objects/storage/urdf/target.urdf (robot description, URDF)
Before this commit: robot target, 1 links, 0 joints
Links:
- link baseLink: geometry collision mesh filename=../obj/target.obj scale=0.0002 0.0002 0.0002; visual mesh filename=../obj/target.obj scale=0.0002 0.0002 0.0002

Commit message: modify objects

File: myGym/envs/objects/geometric/urdf/cube.urdf (robot description, URDF)
Before this commit: robot cube.urdf, 1 links, 0 joints
Links:
- link baseLink: geometry collision mesh filename=./obj/cube.obj scale=.001 .001 .001; visual mesh filename=./obj/cube.obj scale=.001 .001 .001

File: myGym/envs/objects/storage/urdf/target.urdf (robot description, URDF)
Before this commit: robot target, 1 links, 0 joints
Links:
- link baseLink: geometry collision mesh filename=../obj/target.obj scale=0.0005 0.0005 0.0005; visual mesh filename=../obj/target.obj scale=0.0005 0.0005 0.0005

File: myGym/envs/rooms/plane.urdf (robot description, URDF)
Before this commit: robot plane, 1 links, 0 joints
Links:
- link planeLink: mass 0.0 -> 10000.0

Commit message: push task

File: myGym/envs/objects/geometric/urdf/cube.urdf (robot description, URDF)
Before this commit: robot cube.urdf, 1 links, 0 joints
Links:
- link baseLink: geometry collision mesh filename=./obj/cube.obj scale=.0004 .0004 .0004; visual mesh filename=./obj/cube.obj scale=.0004 .0004 .0004

File: myGym/envs/objects/storage/urdf/target.urdf (robot description, URDF)
Before this commit: robot target, 1 links, 0 joints
Links:
- link baseLink: geometry collision mesh filename=../obj/target.obj scale=0.0002 0.0002 0.0002; visual mesh filename=../obj/target.obj scale=0.0002 0.0002 0.0002
