Commit message: update01.06

File: myGym/envs/objects/urdf/cube.urdf (robot description, URDF)
Before this commit: robot cube.urdf, 1 links, 0 joints
Links:
- link baseLink: mass 10 -> 0.01

File: myGym/envs/robots/urdf/niryo_ned2_camera.urdf (robot description, URDF)
Before this commit: robot niryo_ned2, 10 links, 9 joints
Links:
- added link camera_link; visual box size=0.01 0.037 0.037
Joints:
- added joint camera_joint: type fixed, parent wrist_link, child camera_link, origin xyz=0 0.0385 0 rpy=1.5707963268 0 0.174532925199, axis 0 0 1

File: myGym/envs/rooms/urdf/workspace.urdf (robot description, URDF)
Before this commit: robot table, 1 links, 0 joints
Links:
- removed link table
- added link workspace, mass 10.0; collision box size=0.297 0.21 0.001; visual box size=0.297 0.21 0.001
